File: V3-wire-pads/JlinkBreakout.sch (KiCad schematic (older format))
At the start: 15 parts, among them J1 JLINK, J2 TC, J3 SWD, J4 PWR_IN, U1 SGM2019

Commit message: Add LCSC part numbers to resistors
Parts:
- R2: LCSC (none) -> C4184
- R3: LCSC (none) -> C23126
- R4: LCSC (none) -> C23070
Changed lines of the file:
@@
 F 2 "Resistor_SMD:R_0603_1608Metric" V 3730 6300 50  0001 C CNN
 F 3 "~" H 3800 6300 50  0001 C CNN
-F 4 "" V 3800 6300 50  0001 C CNN "LCSC"
+F 4 "C4184" V 3800 6300 50  0001 C CNN "LCSC"
 	1    3800 6300
 	0    1    1    0
@@
 F 2 "Resistor_SMD:R_0603_1608Metric" V 3730 6600 50  0001 C CNN
 F 3 "~" H 3800 6600 50  0001 C CNN
-F 4 "" V 3800 6600 50  0001 C CNN "LCSC"
+F 4 "C23126" V 3800 6600 50  0001 C CNN "LCSC"
 	1    3800 6600
 	0    1    1    0
@@
 F 2 "Resistor_SMD:R_0603_1608Metric" V 3730 6900 50  0001 C CNN
 F 3 "~" H 3800 6900 50  0001 C CNN
-F 4 "" V 3800 6900 50  0001 C CNN "LCSC"
+F 4 "C23070" V 3800 6900 50  0001 C CNN "LCSC"
 	1    3800 6900
 	0    1    1    0
